Commit message: fix

File: lio_sam/config/robot.urdf.xacro (robot description, xacro)
@@ -13,25 +13,25 @@
     <parent link="base_link" />
     <child link="livox_frame" />
-    <origin xyz="0.15 0 0.1" rpy="0 0 0" />
+    <origin xyz="0.13 0 0.19" rpy="0 0 0" />
   </joint>
-  <link name="camera_left_depth_optical_frame"> </link>
-  <joint name="camera_left_joint" type="fixed">
-    <parent link="base_link" />
-    <child link="camera_left_depth_optical_frame" />
-    <origin xyz="0.266842719249179 0.0881830869392123 0.0807512430601606"
-            rpy="-2.00712863979348 0 -1.13446401379631" />
-  </joint>
-  <link name="camera_right_depth_optical_frame"> </link>
-    <joint name="camera_right_joint" type="fixed">
-      <parent link="base_link" />
-      <child link="camera_right_depth_optical_frame" />
-      <origin xyz="0.287973632336214 -0.0428676975873733 0.0807512430601605"
-              rpy="-2.00712863979348 0 -2.00712863979348" />
-    </joint>
-  <link name="navsat_link"> </link>
-  <joint name="navsat_joint" type="fixed">
-    <parent link="base_link" />
-    <child link="navsat_link" />
-    <origin xyz="0 0 0" rpy="0 0 0" />
-  </joint>
+  <!-- <link name="camera_left_depth_optical_frame"> </link> -->
+  <!-- <joint name="camera_left_joint" type="fixed"> -->
+    <!-- <parent link="base_link" /> -->
+    <!-- <child link="camera_left_depth_optical_frame" /> -->
+    <!-- <origin xyz="0.266842719249179 0.0881830869392123 0.0807512430601606"  -->
+            <!-- rpy="-2.00712863979348 0 -1.13446401379631" /> -->
+  <!-- </joint>  -->
+  <!-- <link name="camera_right_depth_optical_frame"> </link> -->
+    <!-- <joint name="camera_right_joint" type="fixed"> -->
+      <!-- <parent link="base_link" /> -->
+      <!-- <child link="camera_right_depth_optical_frame" /> -->
+      <!-- <origin xyz="0.287973632336214 -0.0428676975873733 0.0807512430601605"  -->
+              <!-- rpy="-2.00712863979348 0 -2.00712863979348" /> -->
+    <!-- </joint>  -->
+  <!-- <link name="navsat_link"> </link> -->
+  <!-- <joint name="navsat_joint" type="fixed"> -->
+    <!-- <parent link="base_link" /> -->
+    <!-- <child link="navsat_link" /> -->
+    <!-- <origin xyz="0 0 0" rpy="0 0 0" /> -->
+  <!-- </joint> -->
 </robot>

File: nav2_bringup/urdf/fd_base.xacro (robot description, xacro)
@@ -3,35 +3,49 @@
   <xacro:property name="PI" value="3.1415926535897931" />
   <link name="odom"></link>
-  <link name="base_link"></link>
-  <joint name="base_link_joint" type="fixed">
-    <parent link="odom"/>
-    <child link="base_link" />
-    <origin xyz="0 0 0" rpy="0 0 0" />
-  </joint>
-  <link name="livox_frame"> </link>
-  <joint name="lidar_joint" type="fixed">
-    <parent link="base_link" />
-    <child link="livox_frame" />
-    <origin xyz="0.15 0 0.1" rpy="0 0 0" />
-  </joint>
-  <link name="camera_left_depth_optical_frame"> </link>
-  <joint name="camera_left_joint" type="fixed">
-    <parent link="base_link" />
-    <child link="camera_left_depth_optical_frame" />
-    <origin xyz="0.266842719249179 0.0881830869392123 0.0807512430601606"
-            rpy="-2.00712863979348 0 -1.13446401379631" />
-  </joint>
-  <link name="camera_right_depth_optical_frame"> </link>
-    <joint name="camera_right_joint" type="fixed">
+    <link name="base_link"></link>
+    <joint name="base_link_joint" type="fixed">
+      <parent link="odom"/>
+      <child link="base_link" />
+      <origin xyz="0 0 0" rpy="0 0 0" />
+    </joint>
+    <link name="odom_wheel_link"></link>
+    <joint name="wheel_joint" type="fixed">
+      <parent link="base_link"/>
+      <child link="odom_wheel_link"/>
+      <origin xyz="0 0 0.0845" rpy="0 0 0"/>
+    </joint>
+    <link name="laser_link"> </link>
+    <joint name="lidar_joint" type="fixed">
       <parent link="base_link" />
-      <child link="camera_right_depth_optical_frame" />
-      <origin xyz="0.287973632336214 -0.0428676975873733 0.0807512430601605"
-              rpy="-2.00712863979348 0 -2.00712863979348" />
+      <child link="laser_link" />
+      <origin xyz="0.124 0 0.20142" rpy="0 0 0" />
     </joint>
-  <link name="navsat_link"> </link>
-  <joint name="navsat_joint" type="fixed">
-    <parent link="base_link" />
-    <child link="navsat_link" />
-    <origin xyz="0 0 0" rpy="0 0 0" />
-  </joint>
+    <link name="imu_link"> </link>
+    <joint name="imu_joint" type="fixed">
+      <parent link="laser_link" />
+      <child link="imu_link" />
+      <origin xyz="0.08 0 -0.055" rpy="3.14 0 0" />
+    </joint>
+    <link name="camera_left_depth_optical_frame"> </link>
+    <joint name="camera_left_joint" type="fixed">
+      <parent link="base_link" />
+      <child link="camera_left_depth_optical_frame" />
+      <origin
+        xyz="0.268526757018066 -0.0555348839735371 -0.0214999999778343"
+        rpy="-1.5707963267949 0 -1.83259571459405" />
+    </joint>
+    <link name="camera_right_depth_optical_frame"> </link>
+      <joint name="camera_right_joint" type="fixed">
+        <parent link="base_link" />
+        <child link="camera_right_depth_optical_frame" />
+        <origin
+          xyz="0.268526757018066 0.0555348839735374 -0.0214999999778343"
+          rpy="1.5707963267949 0 1.83259571459405" />
+      </joint>
+    <link name="navsat_link"> </link>
+    <joint name="navsat_joint" type="fixed">
+      <parent link="base_link" />
+      <child link="navsat_link" />
+      <origin xyz="0 0 0" rpy="0 0 0" />
+    </joint>
 </robot>

Commit message: fix

File: lio_sam/config/robot.urdf.xacro (robot description, xacro)
@@ -14,4 +14,20 @@
     <child link="livox_frame" />
     <origin xyz="0.13 0 0.19" rpy="0 0 0" />
+  </joint>
+  <link name="camera_left_depth_optical_frame"> </link>
+  <joint name="camera_left_joint" type="fixed">
+    <parent link="base_link" />
+    <child link="camera_left_depth_optical_frame" />
+    <origin xyz="0.2745 0.04298 0.051" rpy="1.5708 0 2.18167" />
+    <!-- <origin xyz="0.268526757018066 0.0555348839735374 0.064"
+            rpy="1.5707963267949 0 1.83259571459405" /> -->
+  </joint>
+  <link name="camera_right_depth_optical_frame"> </link>
+  <joint name="camera_right_joint" type="fixed">
+    <parent link="base_link" />
+    <child link="camera_right_depth_optical_frame" />
+    <origin xyz="0.2745 -0.04298 0.051" rpy="-1.5708 0 -2.18167" />
+    <!--   <origin xyz="0.268526757018066 -0.055534883973537 0.064"
+              rpy="-1.5707963267949 0 -1.83259571459405" /> -->
   </joint>
   <!-- <link name="camera_left_depth_optical_frame"> </link> -->
